Commit message: 加入感知的代码

File: legged_control/legged_examples/legged_unitree/unitree_description/urdf/go1.urdf (robot description, URDF)
Before this commit: robot robot, 18 links, 17 joints
Links:
- added link livox, mass 0.1; visual mesh filename=package://livox_laser_simulation/meshes/mid360mm.stl
Joints:
- added joint livox_joint: type fixed, parent base, child livox, origin xyz=0.2 0.0 0.1 rpy=0 0 0

File: legged_control/legged_examples/legged_unitree/unitree_description/urdf/robot.xacro (robot description, xacro)
@@ -7,4 +7,6 @@
     <xacro:include filename="$(find unitree_description)/urdf/common/imu.xacro"/>
     <xacro:include filename="$(find unitree_description)/urdf/$(arg robot_type)/const.xacro"/>
+    <xacro:include filename="$(find unitree_description)/urdf/common/laser.xacro"/>
+    <!-- <xacro:include filename="$(find unitree_description)/urdf/livox_mid360.xacro"/> -->
     <!-- <link name="world"/>
     <joint name="base_static_joint" type="fixed">
@@ -35,5 +37,12 @@
         </inertial>
     </link>
+    <joint name="base_joint" type="fixed">
+        <origin xyz="0.0 0.0 0." rpy="0 0 0"/>
+        <parent link="base"/>
+        <child link="base_footprint"/>
+    </joint>
+    <link name="base_footprint"/>
     <xacro:IMU connected_to="base" imu_name="unitree_imu" xyz="0. 0. 0." rpy="0. 0. 0."/>
+    <!-- <xacro:Livox_Mid360 /> -->
     <xacro:leg prefix="RF" mirror="-1" mirror_dae="False" front_hind="1" front_hind_dae="True">
         <origin rpy="0 0 0" xyz="${leg_offset_x} ${-leg_offset_y} 0"/>
